Commit message: Fix tool mesh path

File: iiwa_description/urdf/tool.xacro (robot description, xacro)
@@ -25,5 +25,5 @@
       <origin xyz="0 0 0" rpy="0 0 0"/>
       <geometry>
-	<mesh filename="package://iiwa_tool_description/meshes/visual/tool.stl"/>
+	      <mesh filename="package://iiwa_description/meshes/tool/visual/tool.stl"/>
 	<!-- 	<cylinder length="0.1275" radius="0.020"/> -->
       </geometry>
@@ -33,5 +33,5 @@
       <origin xyz="0 0 0" rpy="0 0 0"/>
       <geometry>
-	<mesh filename="package://iiwa_tool_description/meshes/visual/tool.stl"/>
+	      <mesh filename="package://iiwa_description/meshes/tool/collision/tool.stl"/>
 	<!-- 	<cylinder length="0.1275" radius="0.020"/> -->
       </geometry>
