Commit message: Fix the flange model origin to the geometric center

File: iiwa_description/urdf/flange.xacro (robot description, xacro)
@@ -10,6 +10,6 @@
   <xacro:property name="robot_name" value="iiwa" />
   <xacro:property name="tool_mass" value="0.200" />
-  <xacro:property name="tool_joint_offset" value="0.00 0.00 0.00" />
-  <xacro:property name="tool_link_offset" value="0.00 0.00 0.1275" />
+  <xacro:property name="tool_joint_offset" value="0.0155 0.00 0.0275" />
+  <xacro:property name="tool_link_offset" value="0.00 0.00 0.00" />
   <!--  Here we define a dummy joint between the tip of the iiwa7 and the base of the tool.
   There is no offset between the two, that means the tool is attached at the robot flange. -->

Commit message: For test

File: iiwa_description/urdf/flange.xacro (robot description, xacro)
@@ -10,5 +10,5 @@
   <xacro:property name="robot_name" value="iiwa" />
   <xacro:property name="tool_mass" value="0.200" />
-  <xacro:property name="tool_joint_offset" value="0.0155 0.00 0.0275" />
+  <xacro:property name="tool_joint_offset" value="0.0155 0.00 0.0575" />
   <xacro:property name="tool_link_offset" value="0.00 0.00 0.00" />
   <!--  Here we define a dummy joint between the tip of the iiwa7 and the base of the tool.
