Commit message: Added Texture to IIWA in Gazebo

File: iiwa_description/urdf/iiwa.gazebo.xacro (robot description, xacro)
@@ -22,5 +22,4 @@
     <!-- Link0 -->
     <gazebo reference="${robot_name}_link_0">
-      <material>Gazebo/Grey</material>
       <mu1>0.2</mu1>
       <mu2>0.2</mu2>
@@ -28,5 +27,4 @@
     <!-- Link1 -->
     <gazebo reference="${robot_name}_link_1">
-      <material>Gazebo/Orange</material>
       <mu1>0.2</mu1>
       <mu2>0.2</mu2>
@@ -34,5 +32,4 @@
     <!-- Link2 -->
     <gazebo reference="${robot_name}_link_2">
-      <material>Gazebo/Orange</material>
       <mu1>0.2</mu1>
       <mu2>0.2</mu2>
@@ -40,5 +37,4 @@
     <!-- Link3 -->
     <gazebo reference="${robot_name}_link_3">
-      <material>Gazebo/Orange</material>
       <mu1>0.2</mu1>
       <mu2>0.2</mu2>
@@ -46,5 +42,4 @@
     <!-- Link4 -->
     <gazebo reference="${robot_name}_link_4">
-      <material>Gazebo/Orange</material>
       <mu1>0.2</mu1>
       <mu2>0.2</mu2>
@@ -52,5 +47,4 @@
     <!-- Link5 -->
     <gazebo reference="${robot_name}_link_5">
-      <material>Gazebo/Orange</material>
       <mu1>0.2</mu1>
       <mu2>0.2</mu2>
@@ -58,5 +52,4 @@
     <!-- Link6 -->
     <gazebo reference="${robot_name}_link_6">
-      <material>Gazebo/Orange</material>
       <mu1>0.2</mu1>
       <mu2>0.2</mu2>

File: iiwa_description/urdf/iiwa7.xacro (robot description, xacro)
@@ -29,7 +29,6 @@
         <origin xyz="0 0 0" rpy="0 0 0"/>
         <geometry>
-          <mesh filename="package://iiwa_description/meshes/iiwa7/visual/link_0.stl"/>
-        </geometry>
-        <material name="Grey"/>
+          <mesh filename="package://iiwa_description/meshes/iiwa7/visual/link_0.dae"/>
+        </geometry>
       </visual>
       <collision>
@@ -38,5 +37,4 @@
           <mesh filename="package://iiwa_description/meshes/iiwa7/collision/link_0.stl"/>
         </geometry>
-        <material name="Grey"/>
       </collision>
       <self_collision_checking>
@@ -70,7 +68,6 @@
         <origin xyz="0 0 0.0075" rpy="0 0 0"/>
         <geometry>
-          <mesh filename="package://iiwa_description/meshes/iiwa7/visual/link_1.stl"/>
-        </geometry>
-        <material name="Orange"/>
+          <mesh filename="package://iiwa_description/meshes/iiwa7/visual/link_1.dae"/>
+        </geometry>
       </visual>
       <collision>
@@ -79,5 +76,4 @@
           <mesh filename="package://iiwa_description/meshes/iiwa7/collision/link_1.stl"/>
         </geometry>
-        <material name="Orange"/>
       </collision>
     </link>
@@ -104,7 +100,6 @@
         <origin xyz="0 0 0" rpy="0 0 0"/>
         <geometry>
-          <mesh filename="package://iiwa_description/meshes/iiwa7/visual/link_2.stl"/>
-        </geometry>
-        <material name="Orange"/>
+          <mesh filename="package://iiwa_description/meshes/iiwa7/visual/link_2.dae"/>
+        </geometry>
       </visual>
       <collision>
@@ -113,5 +108,4 @@
           <mesh filename="package://iiwa_description/meshes/iiwa7/collision/link_2.stl"/>
         </geometry>
-        <material name="Orange"/>
       </collision>
     </link>
@@ -138,7 +132,6 @@
         <origin xyz="0 0 -0.026" rpy="0 0 0"/>
         <geometry>
-          <mesh filename="package://iiwa_description/meshes/iiwa7/visual/link_3.stl"/>
-        </geometry>
-        <material name="Orange"/>
+          <mesh filename="package://iiwa_description/meshes/iiwa7/visual/link_3.dae"/>
+        </geometry>
       </visual>
       <collision>
@@ -147,5 +140,4 @@
           <mesh filename="package://iiwa_description/meshes/iiwa7/collision/link_3.stl"/>
         </geometry>
-        <material name="Orange"/>
       </collision>
     </link>
@@ -172,7 +164,6 @@
         <origin xyz="0 0 0" rpy="0 0 0"/>
         <geometry>
-          <mesh filename="package://iiwa_description/meshes/iiwa7/visual/link_4.stl"/>
-        </geometry>
-        <material name="Orange"/>
+          <mesh filename="package://iiwa_description/meshes/iiwa7/visual/link_4.dae"/>
+        </geometry>
       </visual>
       <collision>
@@ -181,5 +172,4 @@
           <mesh filename="package://iiwa_description/meshes/iiwa7/collision/link_4.stl"/>
         </geometry>
-        <material name="Orange"/>
       </collision>
     </link>
@@ -206,7 +196,6 @@
         <origin xyz="0 0 -0.026" rpy="0 0 0"/>
         <geometry>
-          <mesh filename="package://iiwa_description/meshes/iiwa7/visual/link_5.stl"/>
-        </geometry>
-        <material name="Orange"/>
+          <mesh filename="package://iiwa_description/meshes/iiwa7/visual/link_5.dae"/>
+        </geometry>
       </visual>
       <collision>
@@ -215,5 +204,4 @@
           <mesh filename="package://iiwa_description/meshes/iiwa7/collision/link_5.stl"/>
         </geometry>
-        <material name="Orange"/>
       </collision>
     </link>
@@ -240,7 +228,6 @@
         <origin xyz="0 0 0" rpy="0 0 0"/>
         <geometry>
-          <mesh filename="package://iiwa_description/meshes/iiwa7/visual/link_6.stl"/>
-        </geometry>
-        <material name="Orange"/>
+          <mesh filename="package://iiwa_description/meshes/iiwa7/visual/link_6.dae"/>
+        </geometry>
       </visual>
       <collision>
@@ -249,5 +236,4 @@
           <mesh filename="package://iiwa_description/meshes/iiwa7/collision/link_6.stl"/>
         </geometry>
-        <material name="Orange"/>
       </collision>
     </link>

Commit message: Add tool attached model

File: iiwa_description/urdf/iiwa.gazebo.xacro (robot description, xacro)
@@ -61,4 +61,10 @@
       <mu2>0.2</mu2>
     </gazebo>
+    <!-- Tool -->
+    <gazebo reference="tool_link">
+      <material>Gazebo/Grey</material>
+      <mu1>0.2</mu1>
+      <mu2>0.2</mu2>
+    </gazebo>
   </xacro:macro>
 </robot>

Commit message: add camera instead of tool

File: iiwa_description/urdf/iiwa.gazebo.xacro (robot description, xacro)
@@ -61,9 +61,43 @@
       <mu2>0.2</mu2>
     </gazebo>
-    <!-- Tool -->
-    <gazebo reference="tool_link">
-      <material>Gazebo/Grey</material>
-      <mu1>0.2</mu1>
-      <mu2>0.2</mu2>
+    <!-- camera -->
+    <gazebo reference="camera_link">
+      <sensor type="camera" name="camera1">
+        <update_rate>30.0</update_rate>
+        <camera name="head">
+          <horizontal_fov>1.3962634</horizontal_fov>
+          <image>
+            <width>800</width>
+            <height>800</height>
+            <format>R8G8B8</format>
+          </image>
+          <clip>
+            <near>0.02</near>
+            <far>300</far>
+          </clip>
+          <noise>
+            <type>gaussian</type>
+            <!-- Noise is sampled independently per pixel on each frame.
+                That pixel's noise value is added to each of its color
+                channels, which at that point lie in the range [0,1]. -->
+            <mean>0.0</mean>
+            <stddev>0.007</stddev>
+          </noise>
+        </camera>
+        <plugin name="camera_controller" filename="libgazebo_ros_camera.so">
+          <alwaysOn>true</alwaysOn>
+          <updateRate>0.0</updateRate>
+          <cameraName>rrbot/camera1</cameraName>
+          <imageTopicName>image_raw</imageTopicName>
+          <cameraInfoTopicName>camera_info</cameraInfoTopicName>
+          <frameName>camera_link</frameName>
+          <hackBaseline>0.07</hackBaseline>
+          <distortionK1>0.0</distortionK1>
+          <distortionK2>0.0</distortionK2>
+          <distortionK3>0.0</distortionK3>
+          <distortionT1>0.0</distortionT1>
+          <distortionT2>0.0</distortionT2>
+        </plugin>
+      </sensor>
     </gazebo>
   </xacro:macro>
